File: DL/_autosave-DL.kicad_pcb (KiCad board)
At the start: 2 copper layers, 97.8 x 116.8 mm, 39 parts, among them IC1 MCP6V96UT-E_OT, IC2 SCD42-D-R2, IC3 TGS3870-B00, J3 SD_Card, J4 Conn_01x05_Male, J5 Conn_01x05_Male, J6 Conn_01x05_Male, J7 Conn_01x05_Male, Q1 BSS84, Q2 2N7002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

Commit message: PCB layout interation no. 2
Other:
- board size 97.8 x 116.8 mm -> 80.3 x 150.4 mm
Changed lines of the file:
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@@
     )
   )
-  (gr_rect (start 21.59 17.78) (end 119.38 134.62) (layer "Edge.Cuts") (width 0.1) (fill none))
+  (gr_rect (start 21.59 17.78) (end 101.854 168.148) (layer "Edge.Cuts") (width 0.1) (fill none))
   (segment (start 41.91 74.93) (end 41.91 77.47) (width 0.25) (layer "F.Cu") (net 1))
   (segment (start 68.115 115.57) (end 66.04 115.57) (width 0.25) (layer "F.Cu") (net 1))
@@
     (polygon
       (pts
-        (xy 121.412 136.144)
-        (xy 19.304 136.144)
+        (xy 121.412 173.736)
+        (xy 19.304 173.736)
         (xy 20.32 16.51)
         (xy 121.666 15.494)
@@
     (polygon
       (pts
-        (xy 121.412 136.144)
-        (xy 19.304 136.144)
+        (xy 121.412 174.244)
+        (xy 19.304 174.244)
         (xy 20.066 16.51)
         (xy 121.412 15.748)
