File: DL/DL.kicad_pcb (KiCad board)
At the start: 2 copper layers, 97.8 x 116.8 mm, 39 parts, among them IC1 MCP6V96UT-E_OT, IC2 SCD42-D-R2, IC3 TGS3870-B00, J3 SD_Card, J4 Conn_01x05_Male, J5 Conn_01x05_Male, J6 Conn_01x05_Male, J7 Conn_01x05_Male, Q1 BSS84, Q2 2N7002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

Commit message: Add files via upload
Updated pinout 1/2
Parts:
- moved R16 2.52 mm to (45.5, 67.3)
- moved R17 2.52 mm to (45.5, 64.8)
- moved R18 2.52 mm to (45.5, 62.2)
- moved R19 2.52 mm to (45.5, 59.7)
- moved R20 2.52 mm to (45.5, 57.1)
Routing:
- net Net-(J4-Pad5): track 5.08 -> 2.56 mm
- net Net-(J4-Pad4): track 5.08 -> 2.56 mm
- net Net-(J4-Pad3): track 5.08 -> 2.56 mm
- net Net-(J4-Pad2): track 5.08 -> 2.56 mm
- net Net-(J4-Pad1): track 5.08 -> 2.56 mm
- net GP14/SPI_SCK1/I2C_SDA1: track 11.2 -> 13.8 mm
- net GP13/SPI_CSn1/I2C_SCL0/UART_RX0: track 12.3 -> 14.8 mm
- net GP12/SPI_RX1/I2C_SDA0/UART_TX0: track 12.3 -> 14.8 mm
- net GP11/SPI_TX1/I2C_SCL1: track 12.3 -> 14.8 mm
- net GP10/SPI_SCK1/I2C_SDA1: track 12.3 -> 14.8 mm
Other:
- board size 97.8 x 116.8 mm -> 80.3 x 150.4 mm
Changed lines of the file:
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@@
   (net 65 "VBUS")
   (footprint "Resistor_SMD:R_0805_2012Metric_Pad1.20x1.40mm_HandSolder" (layer "F.Cu")
-    (at 47.99 64.77)
+    (at 45.466 64.77)
     (descr "Resistor SMD 0805 (2012 Metric), square (rectangular) end terminal, IPC_7351 nominal with elongated pad for handsoldering. (Body size source: IPC-SM-782 page 72, https://www.pcb-3d.com/wordpress/wp-content/uploads/ipc-sm-782a_amendment_1_and_2.pdf), generated with kicad-footprint-generator")
     (tags "resistor handsolder")
@@
     (fp_arc (start -2.06 0) (mid 2.54 -4.6) (end 7.14 0) (layer "Dwgs.User") (width 0.1))
     (fp_arc (start 7.14 0) (mid 2.54 4.6) (end -2.06 0) (layer "Dwgs.User") (width 0.1))
-    (pad "1" thru_hole rect (at 0 0 90) (size 1.56 1.56) (drill 1.04) (layers *.Cu *.Mask "F.SilkS")
+    (pad "1" thru_hole rect (at 0 0) (size 1.524 3.004) (drill oval 0.762 2.286) (layers *.Cu *.Mask)
       (net 2 "AGND") (pinfunction "COMMON(-)") (pintype "passive"))
-    (pad "2" thru_hole circle (at 2.54 0 90) (size 1.56 1.56) (drill 1.04) (layers *.Cu *.Mask "F.SilkS")
+    (pad "2" thru_hole oval (at 2.54 0) (size 1.524 3.004) (drill oval 0.762 2.286) (layers *.Cu *.Mask)
       (net 23 "GP27{slash}ADC1{slash}I2C_SCL1") (pinfunction "SENSOR_ELECTRODE_(+)") (pintype "passive"))
-    (pad "3" thru_hole circle (at 5.08 0 90) (size 1.56 1.56) (drill 1.04) (layers *.Cu *.Mask "F.SilkS")
+    (pad "3" thru_hole oval (at 5.08 0) (size 1.524 3.004) (drill oval 0.762 2.286) (layers *.Cu *.Mask)
       (net 22 "VD") (pinfunction "HEATER(+)") (pintype "passive"))
   )
@@
   )
   (footprint "Resistor_SMD:R_0805_2012Metric_Pad1.20x1.40mm_HandSolder" (layer "F.Cu")
-    (at 47.99 59.69)
+    (at 45.466 59.69)
     (descr "Resistor SMD 0805 (2012 Metric), square (rectangular) end terminal, IPC_7351 nominal with elongated pad for handsoldering. (Body size source: IPC-SM-782 page 72, https://www.pcb-3d.com/wordpress/wp-content/uploads/ipc-sm-782a_amendment_1_and_2.pdf), generated with kicad-footprint-generator")
     (tags "resistor handsolder")
@@
   )
   (footprint "Resistor_SMD:R_0805_2012Metric_Pad1.20x1.40mm_HandSolder" (layer "F.Cu")
-    (at 47.99 67.31)
+    (at 45.466 67.31)
     (descr "Resistor SMD 0805 (2012 Metric), square (rectangular) end terminal, IPC_7351 nominal with elongated pad for handsoldering. (Body size source: IPC-SM-782 page 72, https://www.pcb-3d.com/wordpress/wp-content/uploads/ipc-sm-782a_amendment_1_and_2.pdf), generated with kicad-footprint-generator")
     (tags "resistor handsolder")
@@
   )
   (footprint "Resistor_SMD:R_0805_2012Metric_Pad1.20x1.40mm_HandSolder" (layer "F.Cu")
-    (at 47.99 57.15)
+    (at 45.466 57.15)
     (descr "Resistor SMD 0805 (2012 Metric), square (rectangular) end terminal, IPC_7351 nominal with elongated pad for handsoldering. (Body size source: IPC-SM-782 page 72, https://www.pcb-3d.com/wordpress/wp-content/uploads/ipc-sm-782a_amendment_1_and_2.pdf), generated with kicad-footprint-generator")
     (tags "resistor handsolder")
@@
   )
   (footprint "Resistor_SMD:R_0805_2012Metric_Pad1.20x1.40mm_HandSolder" (layer "F.Cu")
-    (at 47.99 62.23)
+    (at 45.466 62.23)
     (descr "Resistor SMD 0805 (2012 Metric), square (rectangular) end terminal, IPC_7351 nominal with elongated pad for handsoldering. (Body size source: IPC-SM-782 page 72, https://www.pcb-3d.com/wordpress/wp-content/uploads/ipc-sm-782a_amendment_1_and_2.pdf), generated with kicad-footprint-generator")
     (tags "resistor handsolder")
@@
     )
   )
-  (gr_rect (start 21.59 17.78) (end 119.38 134.62) (layer "Edge.Cuts") (width 0.1) (fill none))
+  (gr_rect (start 21.59 17.78) (end 101.854 168.148) (layer "Edge.Cuts") (width 0.1) (fill none))
   (segment (start 41.91 74.93) (end 41.91 77.47) (width 0.25) (layer "F.Cu") (net 1))
   (segment (start 68.115 115.57) (end 66.04 115.57) (width 0.25) (layer "F.Cu") (net 1))
@@
   (segment (start 47.166 47.044) (end 47.166 50.8) (width 0.25) (layer "F.Cu") (net 27))
   (segment (start 47.166 47.044) (end 47.166 45.798) (width 0.25) (layer "F.Cu") (net 27))
-  (segment (start 46.99 67.31) (end 41.91 67.31) (width 0.25) (layer "F.Cu") (net 32))
-  (segment (start 46.99 64.77) (end 41.91 64.77) (width 0.25) (layer "F.Cu") (net 33))
-  (segment (start 46.99 62.23) (end 41.91 62.23) (width 0.25) (layer "F.Cu") (net 34))
-  (segment (start 46.99 59.69) (end 41.91 59.69) (width 0.25) (layer "F.Cu") (net 35))
-  (segment (start 46.99 57.15) (end 41.91 57.15) (width 0.25) (layer "F.Cu") (net 36))
+  (segment (start 41.91 67.31) (end 44.466 67.31) (width 0.25) (layer "F.Cu") (net 32))
+  (segment (start 41.91 64.77) (end 44.466 64.77) (width 0.25) (layer "F.Cu") (net 33))
+  (segment (start 41.91 62.23) (end 44.466 62.23) (width 0.25) (layer "F.Cu") (net 34))
+  (segment (start 41.91 59.69) (end 44.466 59.69) (width 0.25) (layer "F.Cu") (net 35))
+  (segment (start 41.91 57.15) (end 44.466 57.15) (width 0.25) (layer "F.Cu") (net 36))
   (segment (start 94.996 58.425) (end 88.397 58.425) (width 0.25) (layer "B.Cu") (net 37))
   (segment (start 87.63 58.42) (end 88.392 58.42) (width 0.25) (layer "B.Cu") (net 37))
@@
   (segment (start 82.55 59.69) (end 81.28 58.42) (width 0.25) (layer "F.Cu") (net 47))
   (segment (start 81.28 58.42) (end 77.47 58.42) (width 0.25) (layer "F.Cu") (net 47))
-  (segment (start 55.88 60.96) (end 52.07 64.77) (width 0.25) (layer "F.Cu") (net 48))
-  (segment (start 52.07 64.77) (end 48.99 64.77) (width 0.25) (layer "F.Cu") (net 48))
-  (segment (start 59.69 60.96) (end 55.88 60.96) (width 0.25) (layer "F.Cu") (net 48))
-  (segment (start 55.88 58.42) (end 52.07 62.23) (width 0.25) (layer "F.Cu") (net 49))
-  (segment (start 52.07 62.23) (end 48.99 62.23) (width 0.25) (layer "F.Cu") (net 49))
-  (segment (start 59.69 58.42) (end 55.88 58.42) (width 0.25) (layer "F.Cu") (net 49))
-  (segment (start 55.88 55.88) (end 52.07 59.69) (width 0.25) (layer "F.Cu") (net 50))
-  (segment (start 52.07 59.69) (end 48.99 59.69) (width 0.25) (layer "F.Cu") (net 50))
-  (segment (start 59.69 55.88) (end 55.88 55.88) (width 0.25) (layer "F.Cu") (net 50))
-  (segment (start 55.88 53.34) (end 52.07 57.15) (width 0.25) (layer "F.Cu") (net 51))
-  (segment (start 52.07 57.15) (end 48.99 57.15) (width 0.25) (layer "F.Cu") (net 51))
-  (segment (start 59.69 53.34) (end 55.88 53.34) (width 0.25) (layer "F.Cu") (net 51))
-  (segment (start 50.26 66.04) (end 48.99 67.31) (width 0.25) (layer "F.Cu") (net 52))
-  (segment (start 59.69 66.04) (end 50.26 66.04) (width 0.25) (layer "F.Cu") (net 52))
+  (segment (start 52.07 64.77) (end 55.88 60.96) (width 0.25) (layer "F.Cu") (net 48))
+  (segment (start 55.88 60.96) (end 59.69 60.96) (width 0.25) (layer "F.Cu") (net 48))
+  (segment (start 46.466 64.77) (end 52.07 64.77) (width 0.25) (layer "F.Cu") (net 48))
+  (segment (start 46.466 62.23) (end 52.07 62.23) (width 0.25) (layer "F.Cu") (net 49))
+  (segment (start 55.88 58.42) (end 59.69 58.42) (width 0.25) (layer "F.Cu") (net 49))
+  (segment (start 52.07 62.23) (end 55.88 58.42) (width 0.25) (layer "F.Cu") (net 49))
+  (segment (start 46.466 59.69) (end 52.07 59.69) (width 0.25) (layer "F.Cu") (net 50))
+  (segment (start 52.07 59.69) (end 55.88 55.88) (width 0.25) (layer "F.Cu") (net 50))
+  (segment (start 55.88 55.88) (end 59.69 55.88) (width 0.25) (layer "F.Cu") (net 50))
+  (segment (start 46.466 57.15) (end 52.07 57.15) (width 0.25) (layer "F.Cu") (net 51))
+  (segment (start 55.88 53.34) (end 59.69 53.34) (width 0.25) (layer "F.Cu") (net 51))
+  (segment (start 52.07 57.15) (end 55.88 53.34) (width 0.25) (layer "F.Cu") (net 51))
+  (segment (start 50.26 66.04) (end 59.69 66.04) (width 0.25) (layer "F.Cu") (net 52))
+  (segment (start 48.99 67.31) (end 50.26 66.04) (width 0.25) (layer "F.Cu") (net 52))
+  (segment (start 46.466 67.31) (end 48.99 67.31) (width 0.25) (layer "F.Cu") (net 52))
   (segment (start 59.69 68.58) (end 54.356 73.914) (width 0.25) (layer "F.Cu") (net 59))
   (segment (start 54.356 73.914) (end 54.356 83.82) (width 0.25) (layer "F.Cu") (net 59))
@@
     (connect_pads (clearance 0.508))
     (min_thickness 0.254) (filled_areas_thickness no)
-    (fill (thermal_gap 0.508) (thermal_bridge_width 0.508))
+    (fill yes (thermal_gap 0.508) (thermal_bridge_width 0.508))
     (polygon
       (pts
-        (xy 121.412 136.144)
-        (xy 19.304 136.144)
+        (xy 121.412 173.736)
+        (xy 19.304 173.736)
         (xy 20.32 16.51)
         (xy 121.666 15.494)
@@
     (connect_pads (clearance 0.508))
     (min_thickness 0.254) (filled_areas_thickness no)
-    (fill (thermal_gap 0.508) (thermal_bridge_width 0.508))
+    (fill yes (thermal_gap 0.508) (thermal_bridge_width 0.508))
     (polygon
       (pts
-        (xy 121.412 136.144)
-        (xy 19.304 136.144)
+        (xy 121.412 174.244)
+        (xy 19.304 174.244)
         (xy 20.066 16.51)
         (xy 121.412 15.748)
@@
     )
   )
+  (group "" (id 9e494106-9748-4063-aab8-1d81407059de)
+    (members
+      075d9c19-4714-4a37-add5-ed387775c362
+      1947ea8e-3ea5-493b-ab1c-4e8c5a675398
+      2717f789-6e9a-45e5-ba68-0e97a483a090
+      5e132ece-978a-4ed2-96d2-7bc7057d7641
+      811d06c8-e35a-4323-8e51-11882cc1e2ee
+      9daa9912-e940-4892-aec2-af5c2da81a39
+      bc12d55d-3029-4430-9232-337b1a62028e
+      c82a2eee-3656-406a-a5cb-6b727ac05b34
+      e31ab301-25e2-418f-9cd9-dc83cd2bf700
+      e67ba37b-3be5-45c4-9c11-32a867ec44a3
+      e9015241-3e66-4b19-a676-893935835aee
+    )
+  )

Commit message: Add files via upload
Hopefully last update, use .pretty lib for TGS3870
Parts:
- IC3: footprint TGS3870-B00:TGS3870B00 -> TGS3870B00:TGS3870B00
- moved R16 2.52 mm to (48.0, 67.3)
- moved R17 2.52 mm to (48.0, 64.8)
- moved R18 2.52 mm to (48.0, 62.2)
- moved R19 2.52 mm to (48.0, 59.7)
- moved R20 2.52 mm to (48.0, 57.1)
Routing:
- net Net-(J4-Pad5): track 2.56 -> 5.08 mm
- net Net-(J4-Pad4): track 2.56 -> 5.08 mm
- net Net-(J4-Pad3): track 2.56 -> 5.08 mm
- net Net-(J4-Pad2): track 2.56 -> 5.08 mm
- net Net-(J4-Pad1): track 2.56 -> 5.08 mm
- net GP14/SPI_SCK1/I2C_SDA1: track 13.8 -> 11.2 mm
- net GP13/SPI_CSn1/I2C_SCL0/UART_RX0: track 14.8 -> 12.3 mm
- net GP12/SPI_RX1/I2C_SDA0/UART_TX0: track 14.8 -> 12.3 mm
- net GP11/SPI_TX1/I2C_SCL1: track 14.8 -> 12.3 mm
- net GP10/SPI_SCK1/I2C_SDA1: track 14.8 -> 12.3 mm
